Commit message: Restore old files

File: config/str1ker.urdf (robot description, URDF)
Before this commit: robot str1ker, 13 links, 12 joints
Links:
- removed link solenoid_mount_link
- removed link solenoid_shaft_link
- added link world
- link base_link: mass 0.1 -> 0.70818404
- link drumstick_link: mass 0.091 -> 0.07166651
- link forearm_actuator_body_link: mass 0.199 -> 0.76281631
- link forearm_actuator_connector_link: mass 0.013 -> 0.01257956
- link forearm_actuator_shaft_link: mass 0.113 -> 0.08789688
- link forearm_link: mass 0.703 -> 0.63998399
- link shoulder_link: mass 0.36378108 -> 0.38358403
- link tip_link: mass 0.1 -> None
- link upperarm_actuator_body_link: mass 0.952544 -> 0.70647685
- link upperarm_actuator_shaft_link: mass 0.070 -> 0.04967122
- link upperarm_link: mass 1.139 -> 1.13853115
Joints:
- removed joint solenoid
- removed joint solenoid_mount
- added joint fixed: type fixed, parent world, child base_link, origin xyz=0 0 0 rpy=0 0 0
- joint base: origin xyz=0 0 0 rpy=1.5708 0 0 -> xyz=0 0 0.069 rpy=1.5708 0 0
- joint forearm_actuator_mount: limit lower=-0.146607 upper=-0.118682 effort=100 velocity=1.0 -> lower=-6 upper=6 effort=100 velocity=1.0
- joint upperarm_actuator_mount: limit lower=-1 upper=1 effort=100 velocity=1.0 -> lower=-6 upper=6 effort=100 velocity=1.0
- joint wrist: mimic joint=solenoid multiplier=-6.8966 offset=1.0069 -> (none)
