Commit message: Cleanup configuration

File: config/gazebo_str1ker.urdf (robot description, URDF)
Before this commit: robot str1ker, 13 links, 12 joints
Links:
- removed link world
- added link effector_link, mass 0.001; collision sphere radius=0.02; visual sphere radius=0.02
Joints:
- removed joint fixed
- added joint effector: type fixed, parent forearm_link, child effector_link, origin xyz=-0.02 0.66 0.25 rpy=0 0 0

Commit message: Update moveit config after DH joints

File: config/gazebo_str1ker.urdf (robot description, URDF)
Before this commit: robot str1ker, 13 links, 12 joints
Links:
- removed link effector_link
- added link tip_link, mass 0.1; collision sphere radius=0.01; visual sphere radius=0.01
Joints:
- removed joint effector
- removed joint mount
- added joint base: type revolute, parent base_link, child shoulder_link, origin xyz=0 0 0 rpy=1.5708 0 0, axis 0 1 0, limit lower=-1.4929 upper=1.4929 effort=100 velocity=1.0
- added joint tip: type fixed, parent drumstick_link, child tip_link, origin xyz=0.305 0.0 0.0 rpy=0 0 0
- joint elbow: axis 1 0 0 -> 0 0 1; origin xyz=0 0.4173 0 rpy=0 0 0 -> xyz=0.4173 0 0 rpy=0 0 0
- joint forearm_actuator: axis 0 1 0 -> 1 0 0; origin xyz=0 0.210 0 rpy=0 0 0 -> xyz=0.210 0 0 rpy=0 0 0
- joint forearm_actuator_connector: axis 1 0 0 -> 0 0 1; origin xyz=0 0.0605718 0.004 rpy=0 0 0 -> xyz=0.0605718 0.004 0 rpy=0 0 0
- joint forearm_actuator_mount: axis 1 0 0 -> 0 0 1; origin xyz=0 0.130 -0.034 rpy=0 0 0 -> xyz=0.130 -0.034 0 rpy=0 0 0
- joint shoulder: axis 1 0 0 -> 0 0 1; origin xyz=0 -0.013 0.11518 rpy=0 0 0 -> xyz=-0.013 0.11518 0.0 rpy=0 0 0
- joint solenoid_mount: axis 1 0 0 -> 0 0 1; limit lower=1.25 upper=1.9 effort=100 velocity=1.0 -> lower=-0.09 upper=-0.09 effort=100 velocity=1.0; origin xyz=0.013 0.355 -0.031 rpy=0 0 0 -> xyz=0.355 -0.031 0.013 rpy=0 0 0
- joint upperarm_actuator: axis 0 0 1 -> 1 0 0; origin xyz=0 -0.002 0.153 rpy=0 0 0 -> xyz=0.153 -0.002 0 rpy=0 0 0
- joint upperarm_actuator_mount: axis 1 0 0 -> 0 0 1; limit lower=-0.1 upper=0.1 effort=100 velocity=1.0 -> lower=-1 upper=1 effort=100 velocity=1.0; mimic joint=upperarm_actuator multiplier=0.9 offset=-0.01 -> joint=upperarm_actuator multiplier=0.9 offset=1.560796327; origin xyz=0 0.101045 -0.0504975 rpy=0 0 0 -> xyz=0.101045 -0.0504975 0 rpy=0 0 0
- joint wrist: axis 1 0 0 -> 0 0 1; limit lower=1.0 upper=1.02 effort=100 velocity=1.0 -> lower=0.959931 upper=0.959931 effort=100 velocity=1.0; origin xyz=-0.009 0.48059393086 0 rpy=0 0 0 -> xyz=0.48059393086 0 -0.023 rpy=0 0 0

Commit message: Re-run Move It Setup Assistant to setup Position Control

File: config/gazebo_str1ker.urdf (robot description, URDF)
Before this commit: robot str1ker, 14 links, 13 joints
Joints:
- joint base: limit lower=-1.4929 upper=1.4929 effort=100 velocity=1.0 -> lower=-1.5708 upper=1.5708 effort=100 velocity=3.14160; origin xyz=0 0 0.069 rpy=1.5708 0 0 -> xyz=0 0 0 rpy=1.5708 0 0
- joint fixed: origin xyz=0 0 0 rpy=0 0 0 -> xyz=0 0 0.5 rpy=0 0 0
- joint solenoid: axis 0 0 1 -> 1 0 0
- joint solenoid_mount: type revolute -> fixed
- joint wrist: limit lower=0.959931 upper=0.959931 effort=100 velocity=1.0 -> lower=0.959931 upper=1.0 effort=100 velocity=1.0; mimic (none) -> joint=solenoid multiplier=13.8167 offset=0.9862

Commit message: Fix shoulder offset after re-design

File: config/gazebo_str1ker.urdf (robot description, URDF)
Before this commit: robot str1ker, 14 links, 13 joints
Joints:
- joint shoulder: origin xyz=-0.013 0.11518 0.0 rpy=0 0 0 -> xyz=-0.013 0.109 0.0 rpy=0 0 0
